File: arpeggiator.kicad_sch (KiCad schematic)
At the start: 0 parts

Commit message: add the pitch and sound circuit
Other:
- added sheet 08_reference (schematic/08_reference.kicad_sch)
- added sheet 09_pitch_select (schematic/09_pitch_select.kicad_sch)
- added sheet 10_oscillator (schematic/10_oscillator.kicad_sch)
- added sheet 11_envelope (schematic/11_envelope.kicad_sch)
- added sheet 12_amplifier (schematic/12_amplifier.kicad_sch)
- added sheet 13_line_output (schematic/13_line_output.kicad_sch)
- added sheet 14_analog_power (schematic/14_analog_power.kicad_sch)
- note added: "Analog decoupling and test rails"
- note added: "Arpeggiator"
- note added: "Envelope current source and amplifier"
- note added: "Note and octave voltage selection"
- note added: "Note envelope and stop mute"
- note added: "Oscillator and tuning"
- note added: "Pitch reference and ladder"
- note added: "Sequencer, pitch selection and sound circuit. Main supply, PCB and case are still in progress."
- note added: "Waveform, tone and line output"
- note removed: "Arpeggiator / sequencer circuit"
- note removed: "Circuit in progress. The oscillator, pitch-voltage selection, envelope and main supply are still to be added."

Commit message: add power supply, rail checks and parts list
Other:
- added sheet 15_input_power (schematic/15_input_power.kicad_sch)
- added sheet 16_negative_supply (schematic/16_negative_supply.kicad_sch)
- added sheet 17_negative_monitor (schematic/17_negative_monitor.kicad_sch)
- added sheet 18_input_monitor (schematic/18_input_monitor.kicad_sch)
- added sheet 19_reset_output (schematic/19_reset_output.kicad_sch)
- note added: "12V input and 5V regulator"
- note added: "Analog decoupling"
- note added: "Input voltage check"
- note added: "Negative rail check"
- note added: "Rail reset and output mute"
- note added: "Regulated negative supply"
- note added: "Sequencer, sound and power circuit. PCB layout and case are still in progress."
- note removed: "Analog decoupling and test rails"
- note removed: "Sequencer, pitch selection and sound circuit. Main supply, PCB and case are still in progress."
