File: schematic/04_input_registers.kicad_sch (KiCad schematic)
At the start: 6 parts, among them U201 74HC574, U202 74HC574, U203 74HC574, U204 74HC574, U205 74HC377, U206 74HC377

Commit message: add power supply, rail checks and parts list
Parts:
- U201, U202, U203, U204: MPN (none) -> 74HC574D,653; Manufacturer (none) -> Nexperia; Supplier (none) -> LCSC; Supplier URL (none) -> https://www.lcsc.com/product-detail/C16501.html
- U205, U206: MPN (none) -> 74HC377D,653; Manufacturer (none) -> Nexperia; Supplier (none) -> LCSC; Supplier URL (none) -> https://www.lcsc.com/product-detail/C5639.html
Changed lines of the file:
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@@
       )
     )
-    (property "Datasheet" "http://www.ti.com/lit/gpn/sn74HCT574"
+    (property "Datasheet" "https://assets.nexperia.com/documents/data-sheet/74HC_HCT574.pdf"
       (at 46.989999999999995 46.99000000000001 0.0)
       (effects
@@
         )
         (justify left)
+        (hide yes)
+      )
+    )
+    (property "MPN" "74HC574D,653"
+      (at 64.77 74.93 0.0)
+      (effects
+        (font
+          (size 1.0 1.0)
+        )
+        (hide yes)
+      )
+    )
+    (property "Manufacturer" "Nexperia"
+      (at 64.77 74.93 0.0)
+      (effects
+        (font
+          (size 1.0 1.0)
+        )
+        (hide yes)
+      )
+    )
+    (property "Supplier" "LCSC"
+      (at 64.77 74.93 0.0)
+      (effects
+        (font
+          (size 1.0 1.0)
+        )
+        (hide yes)
+      )
+    )
+    (property "Supplier URL" "https://www.lcsc.com/product-detail/C16501.html"
+      (at 64.77 74.93 0.0)
+      (effects
+        (font
+          (size 1.0 1.0)
+        )
         (hide yes)
       )
@@
       )
     )
-    (property "Datasheet" "http://www.ti.com/lit/gpn/sn74HCT574"
+    (property "Datasheet" "https://assets.nexperia.com/documents/data-sheet/74HC_HCT574.pdf"
       (at 46.989999999999995 157.48 0.0)
       (effects
@@
         )
         (justify left)
+        (hide yes)
+      )
+    )
+    (property "MPN" "74HC574D,653"
+      (at 64.77 185.42 0.0)
+      (effects
+        (font
+          (size 1.0 1.0)
+        )
+        (hide yes)
+      )
+    )
+    (property "Manufacturer" "Nexperia"
+      (at 64.77 185.42 0.0)
+      (effects
+        (font
+          (size 1.0 1.0)
+        )
+        (hide yes)
+      )
+    )
+    (property "Supplier" "LCSC"
+      (at 64.77 185.42 0.0)
+      (effects
+        (font
+          (size 1.0 1.0)
+        )
+        (hide yes)
+      )
+    )
+    (property "Supplier URL" "https://www.lcsc.com/product-detail/C16501.html"
+      (at 64.77 185.42 0.0)
+      (effects
+        (font
+          (size 1.0 1.0)
+        )
         (hide yes)
       )
@@
       )
     )
-    (property "Datasheet" "http://www.ti.com/lit/gpn/sn74LS377"
+    (property "Datasheet" "https://assets.nexperia.com/documents/data-sheet/74HC_HCT377.pdf"
       (at 317.5 46.99000000000001 0.0)
       (effects
@@
         )
         (justify left)
+        (hide yes)
+      )
+    )
+    (property "MPN" "74HC377D,653"
+      (at 335.28 74.93 0.0)
+      (effects
+        (font
+          (size 1.0 1.0)
+        )
+        (hide yes)
+      )
+    )
+    (property "Manufacturer" "Nexperia"
+      (at 335.28 74.93 0.0)
+      (effects
+        (font
+          (size 1.0 1.0)
+        )
+        (hide yes)
+      )
+    )
+    (property "Supplier" "LCSC"
+      (at 335.28 74.93 0.0)
+      (effects
+        (font
+          (size 1.0 1.0)
+        )
+        (hide yes)
+      )
+    )
+    (property "Supplier URL" "https://www.lcsc.com/product-detail/C5639.html"
+      (at 335.28 74.93 0.0)
+      (effects
+        (font
+          (size 1.0 1.0)
+        )
         (hide yes)
       )
@@
       )
     )
-    (property "Datasheet" "http://www.ti.com/lit/gpn/sn74HCT574"
+    (property "Datasheet" "https://assets.nexperia.com/documents/data-sheet/74HC_HCT574.pdf"
       (at 181.60999999999999 46.99000000000001 0.0)
       (effects
@@
         )
         (justify left)
+        (hide yes)
+      )
+    )
+    (property "MPN" "74HC574D,653"
+      (at 199.39 74.93 0.0)
+      (effects
+        (font
+          (size 1.0 1.0)
+        )
+        (hide yes)
+      )
+    )
+    (property "Manufacturer" "Nexperia"
+      (at 199.39 74.93 0.0)
+      (effects
+        (font
+          (size 1.0 1.0)
+        )
+        (hide yes)
+      )
+    )
+    (property "Supplier" "LCSC"
+      (at 199.39 74.93 0.0)
+      (effects
+        (font
+          (size 1.0 1.0)
+        )
+        (hide yes)
+      )
+    )
+    (property "Supplier URL" "https://www.lcsc.com/product-detail/C16501.html"
+      (at 199.39 74.93 0.0)
+      (effects
+        (font
+          (size 1.0 1.0)
+        )
         (hide yes)
       )
@@
       )
     )
-    (property "Datasheet" "http://www.ti.com/lit/gpn/sn74HCT574"
+    (property "Datasheet" "https://assets.nexperia.com/documents/data-sheet/74HC_HCT574.pdf"
       (at 181.60999999999999 157.48 0.0)
       (effects
@@
         )
         (justify left)
+        (hide yes)
+      )
+    )
+    (property "MPN" "74HC574D,653"
+      (at 199.39 185.42 0.0)
+      (effects
+        (font
+          (size 1.0 1.0)
+        )
+        (hide yes)
+      )
+    )
+    (property "Manufacturer" "Nexperia"
+      (at 199.39 185.42 0.0)
+      (effects
+        (font
+          (size 1.0 1.0)
+        )
+        (hide yes)
+      )
+    )
+    (property "Supplier" "LCSC"
+      (at 199.39 185.42 0.0)
+      (effects
+        (font
+          (size 1.0 1.0)
+        )
+        (hide yes)
+      )
+    )
+    (property "Supplier URL" "https://www.lcsc.com/product-detail/C16501.html"
+      (at 199.39 185.42 0.0)
+      (effects
+        (font
+          (size 1.0 1.0)
+        )
         (hide yes)
       )
@@
       )
     )
-    (property "Datasheet" "http://www.ti.com/lit/gpn/sn74LS377"
+    (property "Datasheet" "https://assets.nexperia.com/documents/data-sheet/74HC_HCT377.pdf"
       (at 317.5 157.48 0.0)
       (effects
@@
         (hide yes)
       )
+    )
+    (property "MPN" "74HC377D,653"
+      (at 335.28 185.42 0.0)
+      (effects
+        (font
+          (size 1.0 1.0)
+        )
+        (hide yes)
+      )
+    )
+    (property "Manufacturer" "Nexperia"
+      (at 335.28 185.42 0.0)
+      (effects
+        (font
+          (size 1.0 1.0)
+        )
+        (hide yes)
+      )
+    )
+    (property "Supplier" "LCSC"
+      (at 335.28 185.42 0.0)
+      (effects
+        (font
+          (size 1.0 1.0)
+        )
+        (hide yes)
+      )
+    )
+    (property "Supplier URL" "https://www.lcsc.com/product-detail/C5639.html"
+      (at 335.28 185.42 0.0)
+      (effects
+        (font
+          (size 1.0 1.0)
+        )
+        (hide yes)
+      )
