File: schematic/09_pitch_select.kicad_sch (KiCad schematic)
At the start: 7 parts, among them U501 OPA4192IDR, U502 ADG706BRUZ, U503 74HC4051D

Commit message: add power supply, rail checks and parts list
Parts:
- U501: MPN (none) -> OPA4192IDR; Manufacturer (none) -> Texas Instruments; Supplier (none) -> LCSC; Supplier URL (none) -> https://www.lcsc.com/product-detail/C2057908.html
- U502: MPN (none) -> ADG706BRUZ-REEL7; Manufacturer (none) -> Analog Devices; Supplier (none) -> LCSC; Supplier URL (none) -> https://www.lcsc.com/product-detail/C408400.html
- U503: MPN (none) -> 74HC4051D,653; Manufacturer (none) -> Nexperia; Supplier (none) -> LCSC
Changed lines of the file:
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@@
+      )
+    )
+    (property "MPN" "OPA4192IDR"
+      (at 180.34 209.55 0.0)
+      (effects
+        (font
+          (size 1.0 1.0)
+        )
+        (hide yes)
+      )
+    )
+    (property "Manufacturer" "Texas Instruments"
+      (at 180.34 209.55 0.0)
+      (effects
+        (font
+          (size 1.0 1.0)
+        )
+        (hide yes)
+      )
+    )
+    (property "Supplier" "LCSC"
+      (at 180.34 209.55 0.0)
+      (effects
+        (font
+          (size 1.0 1.0)
+        )
+        (hide yes)
+      )
+    )
+    (property "Supplier URL" "https://www.lcsc.com/product-detail/C2057908.html"
+      (at 180.34 209.55 0.0)
+      (effects
+        (font
+          (size 1.0 1.0)
+        )
+        (hide yes)
       )
     )
@@
       )
     )
+    (property "MPN" "OPA4192IDR"
+      (at 350.52 209.55 0.0)
+      (effects
+        (font
+          (size 1.0 1.0)
+        )
+        (hide yes)
+      )
+    )
+    (property "Manufacturer" "Texas Instruments"
+      (at 350.52 209.55 0.0)
+      (effects
+        (font
+          (size 1.0 1.0)
+        )
+        (hide yes)
+      )
+    )
+    (property "Supplier" "LCSC"
+      (at 350.52 209.55 0.0)
+      (effects
+        (font
+          (size 1.0 1.0)
+        )
+        (hide yes)
+      )
+    )
+    (property "Supplier URL" "https://www.lcsc.com/product-detail/C2057908.html"
+      (at 350.52 209.55 0.0)
+      (effects
+        (font
+          (size 1.0 1.0)
+        )
+        (hide yes)
+      )
+    )
     (instances
       (project "arpeggiator"
@@
       )
     )
+    (property "MPN" "ADG706BRUZ-REEL7"
+      (at 95.25 100.33 0.0)
+      (effects
+        (font
+          (size 1.0 1.0)
+        )
+        (hide yes)
+      )
+    )
+    (property "Manufacturer" "Analog Devices"
+      (at 95.25 100.33 0.0)
+      (effects
+        (font
+          (size 1.0 1.0)
+        )
+        (hide yes)
+      )
+    )
+    (property "Supplier" "LCSC"
+      (at 95.25 100.33 0.0)
+      (effects
+        (font
+          (size 1.0 1.0)
+        )
+        (hide yes)
+      )
+    )
+    (property "Supplier URL" "https://www.lcsc.com/product-detail/C408400.html"
+      (at 95.25 100.33 0.0)
+      (effects
+        (font
+          (size 1.0 1.0)
+        )
+        (hide yes)
+      )
+    )
     (instances
       (project "arpeggiator"
@@
         (hide yes)
       )
+    )
+    (property "MPN" "74HC4051D,653"
+      (at 294.64 100.33 0.0)
+      (effects
+        (font
+          (size 1.0 1.0)
+        )
+        (hide yes)
+      )
+    )
+    (property "Manufacturer" "Nexperia"
+      (at 294.64 100.33 0.0)
+      (effects
+        (font
+          (size 1.0 1.0)
+        )
+        (hide yes)
+      )
+    )
+    (property "Supplier" "LCSC"
+      (at 294.64 100.33 0.0)
+      (effects
+        (font
+          (size 1.0 1.0)
+        )
+        (hide yes)
+      )
