File: schematic/10_oscillator.kicad_sch (KiCad schematic)
At the start: 22 parts, among them U504 AS3340AD

Commit message: add power supply, rail checks and parts list
Parts:
- R531, R532: MPN (none) -> RNCF0805TKT100K; Manufacturer (none) -> Stackpole; Supplier (none) -> DigiKey; Supplier URL (none) -> https://www.digikey.com/en/products/detail/stackpole-electr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
- RV501: footprint (none) -> Potentiometer_THT:Potentiometer_Bourns_3296W_Vertical; MPN (none) -> 3296W-1-501LF; Manufacturer (none) -> Bourns; Supplier (none) -> LCSC
- RV502: footprint (none) -> Potentiometer_THT:Potentiometer_Bourns_3296W_Vertical; MPN (none) -> 3296W-1-103LF; Manufacturer (none) -> Bourns; Supplier (none) -> LCSC
- RV503: footprint (none) -> Potentiometer_THT:Potentiometer_Bourns_3296W_Vertical; MPN (none) -> 3296W-1-203LF; Manufacturer (none) -> Bourns; Supplier (none) -> LCSC
- U504: value AS3340AD -> AS3340A; footprint Package_SO:SOIC-16_3.9x9.9mm_P1.27mm -> Package_DIP:DIP-16_W7.62mm; symbol Arpeggiator:AS3340AD -> Arpeggiator:AS3340A; MPN (none) -> AS3340A; Manufacturer (none) -> ALFA RPAR; Supplier (none) -> Infinite Machinery; Supplier URL (none) -> https://infinitemachinery.com/as3340a
Changed lines of the file:
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@@
   )
   (symbol
-    (lib_id "Arpeggiator:AS3340AD")
+    (lib_id "Arpeggiator:AS3340A")
     (at 199.39 95.25 0.0)
     (unit 1)
@@
       )
     )
-    (property "Value" "AS3340AD"
+    (property "Value" "AS3340A"
       (at 181.60999999999999 69.31 0.0)
       (effects
@@
       )
     )
-    (property "Footprint" "Package_SO:SOIC-16_3.9x9.9mm_P1.27mm"
+    (property "Footprint" "Package_DIP:DIP-16_W7.62mm"
       (at 181.60999999999999 67.31 0.0)
       (effects
@@
         )
         (justify left)
+        (hide yes)
+      )
+    )
+    (property "MPN" "AS3340A"
+      (at 199.39 95.25 0.0)
+      (effects
+        (font
+          (size 1.0 1.0)
+        )
+        (hide yes)
+      )
+    )
+    (property "Manufacturer" "ALFA RPAR"
+      (at 199.39 95.25 0.0)
+      (effects
+        (font
+          (size 1.0 1.0)
+        )
+        (hide yes)
+      )
+    )
+    (property "Supplier" "Infinite Machinery"
+      (at 199.39 95.25 0.0)
+      (effects
+        (font
+          (size 1.0 1.0)
+        )
+        (hide yes)
+      )
+    )
+    (property "Supplier URL" "https://infinitemachinery.com/as3340a"
+      (at 199.39 95.25 0.0)
+      (effects
+        (font
+          (size 1.0 1.0)
+        )
         (hide yes)
       )
@@
       )
     )
+    (property "MPN" "RNCF0805TKT100K"
+      (at 35.56 54.61 0.0)
+      (effects
+        (font
+          (size 1.0 1.0)
+        )
+        (hide yes)
+      )
+    )
+    (property "Manufacturer" "Stackpole"
+      (at 35.56 54.61 0.0)
+      (effects
+        (font
+          (size 1.0 1.0)
+        )
+        (hide yes)
+      )
+    )
+    (property "Supplier" "DigiKey"
+      (at 35.56 54.61 0.0)
+      (effects
+        (font
+          (size 1.0 1.0)
+        )
+        (hide yes)
+      )
+    )
+    (property "Supplier URL" "https://www.digikey.com/en/products/detail/stackpole-electronics-inc/RNCF0805TKT100K/5014562"
+      (at 35.56 54.61 0.0)
+      (effects
+        (font
+          (size 1.0 1.0)
+        )
+        (hide yes)
+      )
+    )
     (instances
       (project "arpeggiator"
@@
       )
     )
+    (property "MPN" "RNCF0805TKT100K"
+      (at 35.56 100.33 0.0)
+      (effects
+        (font
+          (size 1.0 1.0)
+        )
+        (hide yes)
+      )
+    )
+    (property "Manufacturer" "Stackpole"
+      (at 35.56 100.33 0.0)
+      (effects
+        (font
+          (size 1.0 1.0)
+        )
+        (hide yes)
+      )
+    )
+    (property "Supplier" "DigiKey"
+      (at 35.56 100.33 0.0)
+      (effects
+        (font
+          (size 1.0 1.0)
+        )
+        (hide yes)
+      )
+    )
+    (property "Supplier URL" "https://www.digikey.com/en/products/detail/stackpole-electronics-inc/RNCF0805TKT100K/5014562"
+      (at 35.56 100.33 0.0)
+      (effects
+        (font
+          (size 1.0 1.0)
+        )
+        (hide yes)
+      )
+    )
     (instances
       (project "arpeggiator"
@@
       )
     )
-    (property "Footprint" ""
+    (property "Footprint" "Potentiometer_THT:Potentiometer_Bourns_3296W_Vertical"
       (at 314.96 40.64 0.0)
       (effects
@@
       )
     )
-    (property "Datasheet" ""
+    (property "Datasheet" "https://www.bourns.com/docs/product-datasheets/3296.pdf"
       (at 314.96 40.64 0.0)
       (effects
@@
         )
         (justify left)
+        (hide yes)
+      )
+    )
+    (property "MPN" "3296W-1-501LF"
+      (at 345.44 49.53 0.0)
+      (effects
+        (font
+          (size 1.0 1.0)
+        )
+        (hide yes)
+      )
+    )
+    (property "Manufacturer" "Bourns"
+      (at 345.44 49.53 0.0)
+      (effects
+        (font
+          (size 1.0 1.0)
+        )
+        (hide yes)
+      )
+    )
+    (property "Supplier" "LCSC"
+      (at 345.44 49.53 0.0)
+      (effects
+        (font
+          (size 1.0 1.0)
+        )
         (hide yes)
       )
@@
       )
     )
-    (property "Footprint" ""
+    (property "Footprint" "Potentiometer_THT:Potentiometer_Bourns_3296W_Vertical"
       (at 314.96 135.89 0.0)
       (effects
@@
       )
     )
-    (property "Datasheet" ""
+    (property "Datasheet" "https://www.bourns.com/docs/product-datasheets/3296.pdf"
       (at 314.96 135.89 0.0)
       (effects
@@
         )
         (justify left)
+        (hide yes)
+      )
+    )
+    (property "MPN" "3296W-1-103LF"
+      (at 345.44 144.78 0.0)
+      (effects
+        (font
+          (size 1.0 1.0)
+        )
+        (hide yes)
+      )
+    )
+    (property "Manufacturer" "Bourns"
+      (at 345.44 144.78 0.0)
+      (effects
+        (font
+          (size 1.0 1.0)
+        )
+        (hide yes)
+      )
+    )
+    (property "Supplier" "LCSC"
+      (at 345.44 144.78 0.0)
+      (effects
+        (font
+          (size 1.0 1.0)
+        )
         (hide yes)
       )
@@
       )
     )
-    (property "Footprint" ""
+    (property "Footprint" "Potentiometer_THT:Potentiometer_Bourns_3296W_Vertical"
       (at 168.91 200.66000000000003 0.0)
       (effects
@@
       )
     )
-    (property "Datasheet" ""
+    (property "Datasheet" "https://www.bourns.com/docs/product-datasheets/3296.pdf"
       (at 168.91 200.66000000000003 0.0)
       (effects
@@
         (hide yes)
       )
+    )
+    (property "MPN" "3296W-1-203LF"
+      (at 199.39 209.55 0.0)
+      (effects
+        (font
+          (size 1.0 1.0)
+        )
+        (hide yes)
+      )
+    )
+    (property "Manufacturer" "Bourns"
+      (at 199.39 209.55 0.0)
+      (effects
+        (font
+          (size 1.0 1.0)
+        )
+        (hide yes)
+      )
+    )
+    (property "Supplier" "LCSC"
+      (at 199.39 209.55 0.0)
+      (effects
+        (font
+          (size 1.0 1.0)
+        )
+        (hide yes)
+      )
