File: schematic/14_analog_power.kicad_sch (KiCad schematic)
At the start: 15 parts, among them J501 analog test rails only, U501 OPA4192IDR, U602 OPA4192IDR, U603 TL074HIDR, U604 LM13700M/NOPB

Commit message: add power supply, rail checks and parts list
Parts:
- removed J501: analog test rails only, symbol Connector_Generic:Conn_01x03
- U501, U602: MPN (none) -> OPA4192IDR; Manufacturer (none) -> Texas Instruments; Supplier (none) -> LCSC; Supplier URL (none) -> https://www.lcsc.com/product-detail/C2057908.html
- U603: MPN (none) -> TL074HIDR; Manufacturer (none) -> Texas Instruments; Supplier (none) -> LCSC
- U604: MPN (none) -> LM13700M/NOPB; Manufacturer (none) -> Texas Instruments; Supplier (none) -> LCSC
Other:
- note added: "Analog decoupling"
- note added: "Analog decoupling. The negative rail is regulated to -5V after the charge pump."
- note removed: "Analog decoupling and test rails"
- note removed: "Temporary test rails. Main 12V input protection, +5V regulator and negative supply are still to be drawn."
- title: Analog decoupling and test rails -> Analog decoupling
