File: schematic/events.kicad_sch (KiCad schematic)
At the start: 3 parts, among them U301 74HC74, U302 74HC74, U303 74HC74

Commit message: add power supply, rail checks and parts list
Parts:
- U301, U302, U303: MPN (none) -> 74HC74D,653; Manufacturer (none) -> Nexperia; Supplier (none) -> LCSC
