File: schematic/logic_03.kicad_sch (KiCad schematic)
At the start: 4 parts, among them U406 74HC08, U413 74HC08, U414 74HC08, U417 74HC08

Commit message: add power supply, rail checks and parts list
Parts:
- U406, U413, U414, U417: MPN (none) -> 74HC08D,653; Manufacturer (none) -> Nexperia; Supplier (none) -> LCSC
