File: schematic/logic_05.kicad_sch (KiCad schematic)
At the start: 4 parts, among them U407 74HC86, U409 74HC32, U410 74HC32, U415 74HC86

Commit message: add power supply, rail checks and parts list
Parts:
- U407, U415: MPN (none) -> 74HC86D,653; Manufacturer (none) -> Nexperia; Supplier (none) -> LCSC
- U409, U410: MPN (none) -> 74HC32D,653; Manufacturer (none) -> Nexperia; Supplier (none) -> LCSC
