File: schematic/logic_06.kicad_sch (KiCad schematic)
At the start: 4 parts, among them U411 74HC32, U412 74HC32, U419 74HC32, U422 74HC32

Commit message: add power supply, rail checks and parts list
Parts:
- U411, U412, U419, U422: MPN (none) -> 74HC32D,653; Manufacturer (none) -> Nexperia; Supplier (none) -> LCSC
