File: schematic/05_search_counters.kicad_sch (KiCad schematic)
At the start: 7 parts, among them U211 74HC163, U212 74HC138, U213 74HC163, U214 74HC163, U215 74HC163, U216 CD74HC4067M

Commit message: add power supply, rail checks and parts list
Parts:
- U211, U213, U214, U215: MPN (none) -> 74HC163D,653; Manufacturer (none) -> Nexperia; Supplier (none) -> LCSC
- U212: MPN (none) -> 74HC138D,653; Manufacturer (none) -> Nexperia; Supplier (none) -> LCSC
- U216: MPN (none) -> CD74HC4067M; Manufacturer (none) -> Texas Instruments; Supplier (none) -> LCSC
Changed lines of the file:
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@@
       )
     )
-    (property "Datasheet" "http://www.ti.com/lit/gpn/sn74LS163"
+    (property "Datasheet" "https://assets.nexperia.com/documents/data-sheet/74HC_HCT163.pdf"
       (at 46.989999999999995 46.99000000000001 0.0)
       (effects
@@
         )
         (justify left)
+        (hide yes)
+      )
+    )
+    (property "MPN" "74HC163D,653"
+      (at 64.77 74.93 0.0)
+      (effects
+        (font
+          (size 1.0 1.0)
+        )
+        (hide yes)
+      )
+    )
+    (property "Manufacturer" "Nexperia"
+      (at 64.77 74.93 0.0)
+      (effects
+        (font
+          (size 1.0 1.0)
+        )
+        (hide yes)
+      )
+    )
+    (property "Supplier" "LCSC"
+      (at 64.77 74.93 0.0)
+      (effects
+        (font
+          (size 1.0 1.0)
+        )
         (hide yes)
       )
@@
       )
     )
-    (property "Datasheet" "http://www.ti.com/lit/ds/symlink/cd74hc238.pdf"
+    (property "Datasheet" "https://assets.nexperia.com/documents/data-sheet/74HC_HCT138.pdf"
       (at 181.60999999999999 52.07000000000001 0.0)
       (effects
@@
         )
         (justify left)
+        (hide yes)
+      )
+    )
+    (property "MPN" "74HC138D,653"
+      (at 199.39 74.93 0.0)
+      (effects
+        (font
+          (size 1.0 1.0)
+        )
+        (hide yes)
+      )
+    )
+    (property "Manufacturer" "Nexperia"
+      (at 199.39 74.93 0.0)
+      (effects
+        (font
+          (size 1.0 1.0)
+        )
+        (hide yes)
+      )
+    )
+    (property "Supplier" "LCSC"
+      (at 199.39 74.93 0.0)
+      (effects
+        (font
+          (size 1.0 1.0)
+        )
         (hide yes)
       )
@@
       )
     )
-    (property "Datasheet" "http://www.ti.com/lit/gpn/sn74LS163"
+    (property "Datasheet" "https://assets.nexperia.com/documents/data-sheet/74HC_HCT163.pdf"
       (at 46.989999999999995 162.56 0.0)
       (effects
@@
         )
         (justify left)
+        (hide yes)
+      )
+    )
+    (property "MPN" "74HC163D,653"
+      (at 64.77 190.5 0.0)
+      (effects
+        (font
+          (size 1.0 1.0)
+        )
+        (hide yes)
+      )
+    )
+    (property "Manufacturer" "Nexperia"
+      (at 64.77 190.5 0.0)
+      (effects
+        (font
+          (size 1.0 1.0)
+        )
+        (hide yes)
+      )
+    )
+    (property "Supplier" "LCSC"
+      (at 64.77 190.5 0.0)
+      (effects
+        (font
+          (size 1.0 1.0)
+        )
         (hide yes)
       )
@@
       )
     )
-    (property "Datasheet" "http://www.ti.com/lit/gpn/sn74LS163"
+    (property "Datasheet" "https://assets.nexperia.com/documents/data-sheet/74HC_HCT163.pdf"
       (at 181.60999999999999 162.56 0.0)
       (effects
@@
         )
         (justify left)
+        (hide yes)
+      )
+    )
+    (property "MPN" "74HC163D,653"
+      (at 199.39 190.5 0.0)
+      (effects
+        (font
+          (size 1.0 1.0)
+        )
+        (hide yes)
+      )
+    )
+    (property "Manufacturer" "Nexperia"
+      (at 199.39 190.5 0.0)
+      (effects
+        (font
+          (size 1.0 1.0)
+        )
+        (hide yes)
+      )
+    )
+    (property "Supplier" "LCSC"
+      (at 199.39 190.5 0.0)
+      (effects
+        (font
+          (size 1.0 1.0)
+        )
         (hide yes)
       )
@@
       )
     )
-    (property "Datasheet" "http://www.ti.com/lit/gpn/sn74LS163"
+    (property "Datasheet" "https://assets.nexperia.com/documents/data-sheet/74HC_HCT163.pdf"
       (at 317.5 162.56 0.0)
       (effects
@@
         )
         (justify left)
+        (hide yes)
+      )
+    )
+    (property "MPN" "74HC163D,653"
+      (at 335.28 190.5 0.0)
+      (effects
+        (font
+          (size 1.0 1.0)
+        )
+        (hide yes)
+      )
+    )
+    (property "Manufacturer" "Nexperia"
+      (at 335.28 190.5 0.0)
+      (effects
+        (font
+          (size 1.0 1.0)
+        )
+        (hide yes)
+      )
+    )
+    (property "Supplier" "LCSC"
+      (at 335.28 190.5 0.0)
+      (effects
+        (font
+          (size 1.0 1.0)
+        )
         (hide yes)
       )
@@
       )
     )
-    (property "Datasheet" "http://www.ti.com/lit/ds/symlink/cd74hc4067.pdf"
+    (property "Datasheet" "https://www.ti.com/lit/ds/symlink/cd74hc4067.pdf"
       (at 317.5 41.91000000000001 0.0)
       (effects
@@
         (hide yes)
       )
+    )
+    (property "MPN" "CD74HC4067M"
+      (at 335.28 74.93 0.0)
+      (effects
+        (font
+          (size 1.0 1.0)
+        )
+        (hide yes)
+      )
+    )
+    (property "Manufacturer" "Texas Instruments"
+      (at 335.28 74.93 0.0)
+      (effects
+        (font
+          (size 1.0 1.0)
+        )
+        (hide yes)
+      )
+    )
+    (property "Supplier" "LCSC"
+      (at 335.28 74.93 0.0)
+      (effects
+        (font
+          (size 1.0 1.0)
+        )
+        (hide yes)
+      )

Commit message: parts and cheaper PCB files
Parts:
- U211, U213, U214, U215: MPN 74HC163D,653 -> SN74HC163DR; Manufacturer Nexperia -> TI
Changed lines of the file:
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@@
       )
     )
-    (property "MPN" "74HC163D,653"
+    (property "MPN" "SN74HC163DR"
       (at 64.77 74.93 0.0)
       (effects
@@
       )
     )
-    (property "Manufacturer" "Nexperia"
+    (property "Manufacturer" "TI"
       (at 64.77 74.93 0.0)
       (effects
@@
       )
     )
-    (property "MPN" "74HC163D,653"
+    (property "MPN" "SN74HC163DR"
       (at 64.77 190.5 0.0)
       (effects
@@
       )
     )
-    (property "Manufacturer" "Nexperia"
+    (property "Manufacturer" "TI"
       (at 64.77 190.5 0.0)
       (effects
@@
       )
     )
-    (property "MPN" "74HC163D,653"
+    (property "MPN" "SN74HC163DR"
       (at 199.39 190.5 0.0)
       (effects
@@
       )
     )
-    (property "Manufacturer" "Nexperia"
+    (property "Manufacturer" "TI"
       (at 199.39 190.5 0.0)
       (effects
@@
       )
     )
-    (property "MPN" "74HC163D,653"
+    (property "MPN" "SN74HC163DR"
       (at 335.28 190.5 0.0)
       (effects
@@
       )
     )
-    (property "Manufacturer" "Nexperia"
+    (property "Manufacturer" "TI"
       (at 335.28 190.5 0.0)
       (effects
