File: schematic/12_amplifier.kicad_sch (KiCad schematic)
At the start: 18 parts, among them Q606 MMBT3906, U602 OPA4192IDR, U604 LM13700M/NOPB

Commit message: add power supply, rail checks and parts list
Parts:
- D601: MPN (none) -> BAT54GW,115; Manufacturer (none) -> Nexperia; Supplier (none) -> LCSC
- Q606: MPN (none) -> MMBT3906,215; Manufacturer (none) -> Nexperia; Supplier (none) -> LCSC
- R621, R624: MPN (none) -> RNCF0805TKY10K0; Manufacturer (none) -> Stackpole; Supplier (none) -> Mouser; Supplier URL (none) -> https://www.mouser.com/ProductDetail/SEI-Stackpole/RNCF0805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
- R622, R623: MPN (none) -> RNCF0805TKT100K; Manufacturer (none) -> Stackpole; Supplier (none) -> DigiKey; Supplier URL (none) -> https://www.digikey.com/en/products/detail/stackpole-electr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
- RV602: footprint (none) -> Potentiometer_THT:Potentiometer_Bourns_3296W_Vertical; MPN (none) -> 3296W-1-104LF; Manufacturer (none) -> Bourns; Supplier (none) -> LCSC
- U602: MPN (none) -> OPA4192IDR; Manufacturer (none) -> Texas Instruments; Supplier (none) -> LCSC; Supplier URL (none) -> https://www.lcsc.com/product-detail/C2057908.html
- U604: MPN (none) -> LM13700M/NOPB; Manufacturer (none) -> Texas Instruments; Supplier (none) -> LCSC

Commit message: parts and cheaper PCB files
Parts:
- D601: MPN BAT54GW,115 -> BAT54GWX
Changed lines of the file:
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@@
       )
     )
-    (property "MPN" "BAT54GW,115"
+    (property "MPN" "BAT54GWX"
       (at 384.81 100.33 0.0)
       (effects
